Commit message: update README

File: description/jaka/right_jaka.urdf (robot description, URDF)
Before this commit: robot jaka, 8 links, 7 joints
Links:
- link LINK_1: geometry collision mesh filename=package://MoveTo/description/jaka/meshes/LINK_1.STL; visual mesh filename=package://MoveTo/description/jaka/meshes/LINK_1.STL
- link LINK_2: geometry collision mesh filename=package://MoveTo/description/jaka/meshes/LINK_2.STL; visual mesh filename=package://MoveTo/description/jaka/meshes/LINK_2.STL
- link LINK_3: geometry collision mesh filename=package://MoveTo/description/jaka/meshes/LINK_3.STL; visual mesh filename=package://MoveTo/description/jaka/meshes/LINK_3.STL
- link LINK_4: geometry collision mesh filename=package://MoveTo/description/jaka/meshes/LINK_4.STL; visual mesh filename=package://MoveTo/description/jaka/meshes/LINK_4.STL
- link LINK_5: geometry collision mesh filename=package://MoveTo/description/jaka/meshes/LINK_5.STL; visual mesh filename=package://MoveTo/description/jaka/meshes/LINK_5.STL
- link LINK_6: geometry collision mesh filename=package://MoveTo/description/jaka/meshes/LINK_6.STL; visual mesh filename=package://MoveTo/description/jaka/meshes/LINK_6.STL
- link LINK_7: geometry collision mesh filename=package://MoveTo/description/jaka/meshes/LINK_7.STL; visual mesh filename=package://MoveTo/description/jaka/meshes/LINK_7.STL
- link LINK_BASE: geometry collision mesh filename=package://MoveTo/description/jaka/meshes/LINK_BASE.STL; visual mesh filename=package://MoveTo/description/jaka/meshes/LINK_BASE.STL

File: description/jaka/right_jaka_renamed.urdf (robot description, URDF)
Before this commit: robot jaka, 8 links, 7 joints
Links:
- link LINK_1: geometry collision mesh filename=/home/tengxun/lab/pinocchio_ws/src/MoveTo/description/jaka/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; visual mesh filename=/home/tengxun/lab/pinocchio_ws/src/MoveTo/description/jaka/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
- link LINK_2: geometry collision mesh filename=/home/tengxun/lab/pinocchio_ws/src/MoveTo/description/jaka/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; visual mesh filename=/home/tengxun/lab/pinocchio_ws/src/MoveTo/description/jaka/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
- link LINK_3: geometry collision mesh filename=/home/tengxun/lab/pinocchio_ws/src/MoveTo/description/jaka/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; visual mesh filename=/home/tengxun/lab/pinocchio_ws/src/MoveTo/description/jaka/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
- link LINK_4: geometry collision mesh filename=/home/tengxun/lab/pinocchio_ws/src/MoveTo/description/jaka/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; visual mesh filename=/home/tengxun/lab/pinocchio_ws/src/MoveTo/description/jaka/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
- link LINK_5: geometry collision mesh filename=/home/tengxun/lab/pinocchio_ws/src/MoveTo/description/jaka/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; visual mesh filename=/home/tengxun/lab/pinocchio_ws/src/MoveTo/description/jaka/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
- link LINK_6: geometry collision mesh filename=/home/tengxun/lab/pinocchio_ws/src/MoveTo/description/jaka/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; visual mesh filename=/home/tengxun/lab/pinocchio_ws/src/MoveTo/description/jaka/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
- link LINK_7: geometry collision mesh filename=/home/tengxun/lab/pinocchio_ws/src/MoveTo/description/jaka/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; visual mesh filename=/home/tengxun/lab/pinocchio_ws/src/MoveTo/description/jaka/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
- link LINK_BASE: geometry collision mesh filename=/home/tengxun/lab/pinocchio_ws/src/MoveTo/description/jaka/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; visual mesh filename=/home/tengxun/lab/pinocchio_ws/src/MoveTo/description/jaka/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

Commit message: update

File: description/jaka/right_jaka.urdf (robot description, URDF)
Before this commit: robot jaka, 8 links, 7 joints
Links:
- link LINK_1: geometry collision mesh filename=package://OBVP_Planner/description/jaka/meshes/LINK_1.STL; visual mesh filename=package://OBVP_Planner/description/jaka/meshes/LINK_1.STL
- link LINK_2: geometry collision mesh filename=package://OBVP_Planner/description/jaka/meshes/LINK_2.STL; visual mesh filename=package://OBVP_Planner/description/jaka/meshes/LINK_2.STL
- link LINK_3: geometry collision mesh filename=package://OBVP_Planner/description/jaka/meshes/LINK_3.STL; visual mesh filename=package://OBVP_Planner/description/jaka/meshes/LINK_3.STL
- link LINK_4: geometry collision mesh filename=package://OBVP_Planner/description/jaka/meshes/LINK_4.STL; visual mesh filename=package://OBVP_Planner/description/jaka/meshes/LINK_4.STL
- link LINK_5: geometry collision mesh filename=package://OBVP_Planner/description/jaka/meshes/LINK_5.STL; visual mesh filename=package://OBVP_Planner/description/jaka/meshes/LINK_5.STL
- link LINK_6: geometry collision mesh filename=package://OBVP_Planner/description/jaka/meshes/LINK_6.STL; visual mesh filename=package://OBVP_Planner/description/jaka/meshes/LINK_6.STL
- link LINK_7: geometry collision mesh filename=package://OBVP_Planner/description/jaka/meshes/LINK_7.STL; visual mesh filename=package://OBVP_Planner/description/jaka/meshes/LINK_7.STL
- link LINK_BASE: geometry collision mesh filename=package://OBVP_Planner/description/jaka/meshes/LINK_BASE.STL; visual mesh filename=package://OBVP_Planner/description/jaka/meshes/LINK_BASE.STL
